File: Temperature_PCB.kicad_sch (KiCad schematic)
At the start: 30 parts, among them J1 Temp, K1 HF115F/024-1H3B, Q1 2N7002, U2 LM393, U5 AMS1117-5.0

Commit message: VER1.0: плата разведена, файлы для производства готовы
Parts:
- removed J1: Temp, symbol Connector_Generic:Conn_01x03
- removed TH1: Thermistor_NTC_3Wire, Resistor_SMD:R_1206_3216Metric_Pad1.30x1.75mm_HandSolder, symbol Device:Thermistor_NTC_3Wire
- added C5, C6: 100n, Capacitor_SMD:C_0805_2012Metric_Pad1.18x1.45mm_HandSolder, symbol Device:C_Small
- added D3: Logo, Logo_My:Logo_Company_2, symbol Logo_my:Logo_template
- added H1, H2, H3, H4: MountingHole, MountingHole:MountingHole_4.3mm_M4, symbol Mechanical:MountingHole
- added J1: (no value), Connector_Molex:Molex_Mini-Fit_Jr_5569-04A2_2x02_P4.20mm_Horizontal, symbol Connector_Generic:Conn_02x02_Odd_Even
- added J2, J3, J4: (no value), Connector_Molex:Molex_Mini-Fit_Jr_5569-02A2_2x01_P4.20mm_Horizontal, symbol Connector_Generic:Conn_01x02
- added R16, R5: 0, Resistor_SMD:R_0805_2012Metric_Pad1.20x1.40mm_HandSolder, symbol Device:R_Small
- added RV1, RV2: (no value), Potentiometer_my:3362P_1, symbol Device:R_Potentiometer
- added TH1: Thermistor_NTC, Resistor_SMD:R_1206_3216Metric_Pad1.30x1.75mm_HandSolder, symbol Device:Thermistor_NTC
- C2, C3: Description P/N (none) -> Capacitor SMD 50V
- C4: Description P/N (none) -> Capacitor Tantalum SMD; Product Name (none) -> CA45-A010K226T
- C49: Description P/N (none) -> Capacitor Tantalum SMD; Product Name (none) -> CA45-A010K106T
- C50, C53: Description P/N Capacitor SMD 25+V -> Capacitor SMD 50V
- D1: value CD4011 -> (none); Product Name (none) -> CD4011
- D2: value K7809-500R3 -> (none); Product Name (none) -> K7809-500R3
- D28, D5, D6: Purpose PWR -> (none)
- D4: value 1N4007[M7] -> (none); Product Name (none) -> 1N4007[M7]
- K1: value HF115F/024-1H3B -> (none); Product Name (none) -> HF115F/024-1H3B
- Q1: value 2N7002 -> (none); Product Name (none) -> 2N7002
- R10, R11, R4, R6, R8: Description P/N (none) -> Resistor SMD
- R12, R13: Description P/N (none) -> Resistor SMD; Product Name (none) -> RT0805BRD0751RL
- R14, R15: Product Name (none) -> Resistor SMD
- R7: value 20 -> 49.9; Description P/N (none) -> Resistor SMD; Product Name (none) -> RT0805BRD0749R9L
- R9: value 49.9 -> 330; Description P/N (none) -> Resistor SMD; Product Name (none) -> ERA6AEB331V
- U2: value LM393 -> (none); Product Name (none) -> LM393
- U5: value AMS1117-5.0 -> (none); Product Name (none) -> AMS1117-5.0
Connections:
- net +24V: now also J2.2 (Pin_2)
- net GND: now also J1.3 (Pin_3), J2.1 (Pin_1), R16.1, TH1.2; no longer R12.1, R13.1
- net at R8.1, R9.2, U2.5 (+): now also RV2.1
- net at U2.3 (+), U2.6 (-): now also C5.2, C6.2, J1.2 (Pin_2), R5.1, TH1.1; no longer R4.1
- net at R12.2, R7.1: now also RV1.2, RV1.3
- net at R6.1, R7.2, U2.2 (-): now also RV1.1
- net at R13.2, R9.1: now also RV2.2, RV2.3
- net A_IN: now reaches K1.11
- net A_IN: now also K1.21, J3.2 (Pin_2)
- net A_OUT: now reaches K1.14
- net A_OUT: now also K1.24, J4.2 (Pin_2)
- new net: J1.1 (Pin_1), R4.1, R5.2
- new net: C5.1, C6.1, J1.4 (Pin_4), R12.1, R13.1, R16.2
- new net N: J3.1 (Pin_1), J4.1 (Pin_1)
Other:
- note added: "Уставка +13"
- note added: "Уставка +5"
- moved on the sheet: C2, C3, C4, C49, C50, C53, D1, D2, D28, D4, D5, D6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
