File: Temperature_PCB.kicad_sch (KiCad schematic)
At the start: 44 parts

Commit message: VER1.0: обновил гербера и BOM
Parts:
- C4, C49: Description P/N Capacitor Tantalum SMD -> Capacitor Tantalum SMD 10V
- D1: Description P/N (none) -> NAND
- D2: footprint MORNSUN:K78xx-500R3 ÕýÊä³ö -> MORNSUN:K78xx-500R3; Description P/N (none) -> DCDC
- D4: Description P/N (none) -> Diode
- J1, J2, J3, J4: Description P/N (none) -> Connector
- K1: Description P/N (none) -> Relay
- Q1: Description P/N (none) -> MOSFET
- R10, R11, R16, R38, R4, R5, R6, R8: Description P/N Resistor SMD -> Resistor SMD 1%
- R12, R13, R7, R9: Description P/N Resistor SMD -> Resistor SMD 0.1%
- R14, R15: Description P/N Resistor SMD -> Resistor SMD 1%; Product Name Resistor SMD -> (none)
- RV1, RV2: Description P/N (none) -> Potentiometer
- TH1: Description P/N (none) -> Thermistor SMD
- U2: Description P/N (none) -> Op-Amp
- U5: Description P/N (none) -> Linear regulator
Changed lines of the file:
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@@
 			)
 		)
+		(property "Description P/N" "Op-Amp"
+			(at 193.04 184.15 0)
+			(hide yes)
+			(show_name no)
+			(do_not_autoplace no)
+			(effects
+				(font
+					(size 1.27 1.27)
+				)
+			)
+		)
 		(pin "6"
 		)
@@
 			)
 		)
-		(property "Description P/N" "Resistor SMD"
+		(property "Description P/N" "Resistor SMD 1%"
 			(at 109.22 138.43 0)
 			(hide yes)
@@
 			)
 		)
-		(property "Description P/N" "Resistor SMD"
+		(property "Description P/N" "Resistor SMD 1%"
 			(at 194.31 63.5 0)
 			(hide yes)
@@
 			)
 		)
-		(property "Description P/N" ""
+		(property "Description P/N" "Connector"
 			(at 311.15 167.64 0)
 			(hide yes)
@@
 			)
 		)
-		(property "Description P/N" "Resistor SMD"
+		(property "Description P/N" "Resistor SMD 1%"
 			(at 175.26 176.53 0)
 			(hide yes)
@@
 			)
 		)
-		(property "Description P/N" ""
+		(property "Description P/N" "Connector"
 			(at 311.15 180.34 0)
 			(hide yes)
@@
 			)
 		)
-		(property "Description P/N" "Capacitor Tantalum SMD"
+		(property "Description P/N" "Capacitor Tantalum SMD 10V"
 			(at 153.67 67.31 0)
 			(hide yes)
@@
 			)
 		)
-		(property "Description P/N" "Resistor SMD"
+		(property "Description P/N" "Resistor SMD 1%"
 			(at 118.11 63.5 0)
 			(hide yes)
@@
 			)
 		)
-		(property "Product Name" "Resistor SMD"
+		(property "Product Name" ""
 			(at 118.11 63.5 0)
 			(hide yes)
@@
 			)
 		)
-		(property "Description P/N" "Resistor SMD"
+		(property "Description P/N" "Resistor SMD 1%"
 			(at 261.62 133.35 0)
 			(hide yes)
@@
 			)
 		)
-		(property "Product Name" "Resistor SMD"
+		(property "Product Name" ""
 			(at 261.62 133.35 0)
 			(show_name no)
@@
 			)
 		)
-		(property "Footprint" "MORNSUN:K78xx-500R3 ÕýÊä³ö"
+		(property "Footprint" "MORNSUN:K78xx-500R3"
 			(at 135.89 66.04 0)
 			(hide yes)
@@
 			)
 		)
+		(property "Description P/N" "DCDC"
+			(at 140.97 59.69 0)
+			(hide yes)
+			(show_name no)
+			(do_not_autoplace no)
+			(effects
+				(font
+					(size 1.27 1.27)
+				)
+			)
+		)
+		(property "Replacement" ""
+			(at 140.97 59.69 0)
+			(hide yes)
+			(show_name no)
+			(do_not_autoplace no)
+			(effects
+				(font
+					(size 1.27 1.27)
+				)
+			)
+		)
+		(property "Function" ""
+			(at 140.97 59.69 0)
+			(hide yes)
+			(show_name no)
+			(do_not_autoplace no)
+			(effects
+				(font
+					(size 1.27 1.27)
+				)
+			)
+		)
 		(pin "1"
 		)
@@
 			)
 		)
+		(property "Description P/N" "Op-Amp"
+			(at 193.04 146.05 0)
+			(hide yes)
+			(show_name no)
+			(do_not_autoplace no)
+			(effects
+				(font
+					(size 1.27 1.27)
+				)
+			)
+		)
 		(pin "6"
 		)
@@
 			)
 		)
+		(property "Description P/N" "Op-Amp"
+			(at 196.85 115.57 0)
+			(hide yes)
+			(show_name no)
+			(do_not_autoplace no)
+			(effects
+				(font
+					(size 1.27 1.27)
+				)
+			)
+		)
 		(pin "6"
 		)
@@
 			)
 		)
-		(property "Description P/N" "Capacitor Tantalum SMD"
+		(property "Description P/N" "Capacitor Tantalum SMD 10V"
 			(at 182.88 67.31 0)
 			(hide yes)
@@
 			)
 		)
-		(property "Description P/N" "Resistor SMD"
+		(property "Description P/N" "Resistor SMD 1%"
 			(at 115.57 163.83 0)
 			(hide yes)
@@
 			)
 		)
-		(property "Description P/N" ""
+		(property "Description P/N" "Connector"
 			(at 114.3 154.94 0)
 			(hide yes)
@@
 			)
 		)
-		(property "Description P/N" "Resistor SMD"
+		(property "Description P/N" "Resistor SMD 1%"
 			(at 205.74 177.8 0)
 			(hide yes)
@@
 			)
 		)
-		(property "Description P/N" "Resistor SMD"
+		(property "Description P/N" "Resistor SMD 0.1%"
 			(at 175.26 153.67 0)
 			(hide yes)
@@
 			)
 		)
-		(property "Description P/N" "Resistor SMD"
+		(property "Description P/N" "Resistor SMD 1%"
 			(at 205.74 139.7 0)
 			(hide yes)
@@
 			)
 		)
-		(property "Description P/N" "Resistor SMD"
+		(property "Description P/N" "Resistor SMD 0.1%"
 			(at 175.26 158.75 0)
 			(hide yes)
@@
 			)
 		)
-		(property "Description P/N" ""
+		(property "Description P/N" "Thermistor SMD"
 			(at 133.35 148.59 0)
 			(hide yes)
@@
 			)
 		)
+		(property "Description P/N" "NAND"
+			(at 231.14 144.78 0)
+			(hide yes)
+			(show_name no)
+			(do_not_autoplace no)
+			(effects
+				(font
+					(size 1.27 1.27)
+				)
+			)
+		)
 		(pin "9"
 		)
@@
 			)
 		)
-		(property "Description P/N" "Resistor SMD"
+		(property "Description P/N" "Resistor SMD 1%"
 			(at 175.26 138.43 0)
 			(hide yes)
@@
 			)
 		)
-		(property "Description P/N" ""
+		(property "Description P/N" "Connector"
 			(at 104.14 67.31 0)
 			(hide yes)
@@
 			)
 		)
-		(property "Description P/N" "Resistor SMD"
+		(property "Description P/N" "Resistor SMD 0.1%"
 			(at 175.26 196.85 0)
 			(hide yes)
@@
 			)
 		)
+		(property "Description P/N" "MOSFET"
+			(at 259.08 156.21 0)
+			(hide yes)
+			(show_name no)
+			(do_not_autoplace no)
+			(effects
+				(font
+					(size 1.27 1.27)
+				)
+			)
+		)
 		(pin "1"
 		)
@@
 			)
 		)
-		(property "Description P/N" ""
+		(property "Description P/N" "Potentiometer"
 			(at 167.64 191.77 0)
 			(hide yes)
@@
 			)
 		)
+		(property "Description P/N" "Diode"
+			(at 288.29 130.81 0)
+			(hide yes)
+			(show_name no)
+			(do_not_autoplace no)
+			(effects
+				(font
+					(size 1.27 1.27)
+				)
+			)
+		)
 		(pin "2"
 		)
@@
 			)
 		)
-		(property "Description P/N" ""
+		(property "Description P/N" "Potentiometer"
 			(at 167.64 153.67 0)
 			(hide yes)
@@
 			)
 		)
+		(property "Description P/N" "Linear regulator"
+			(at 172.72 63.5 0)
+			(hide yes)
+			(show_name no)
+			(do_not_autoplace no)
+			(effects
+				(font
+					(size 1.27 1.27)
+				)
+			)
+		)
 		(pin "1"
 		)
@@
 			)
 		)
-		(property "Description P/N" ""
+		(property "Description P/N" "Relay"
 			(at 288.29 149.86 0)
 			(hide yes)
@@
 			)
 		)
-		(property "Description P/N" "Resistor SMD"
+		(property "Description P/N" "Resistor SMD 1%"
 			(at 115.57 143.51 0)
 			(hide yes)
@@
 			)
 		)
-		(property "Description P/N" "Resistor SMD"
+		(property "Description P/N" "Resistor SMD 0.1%"
 			(at 175.26 191.77 0)
 			(hide yes)
